File: LAM-4I4O/hardware/LAM-4I4O-REVC/LAM-4I4O-REVC.kicad_pcb (KiCad board)
At the start: 2 copper layers, 65 x 80 mm, 67 parts, among them J1 MC1,5 2G-3.81, J10 MC 1,5/2G-3,81, J11 MC 1,5/2G-3,81, J12 MC 1,5/2G-3,81, J2 MC1,5 2G-3.81, J3 MC1,5 2G-3.81, J4 PLS, J5 MC 1,5/2G-3,81, J6 MC 1,5/2G-3,81, J7 MC 1,5/2G-3,81, J8 MC 1,5/2G-3,81, J9 MC 1,5/2G-3,81, U1 CH32V003AxMx, U2 SN75176BDR, U3 LT1117-5.0, U4 ULN2003

Commit message: fix(LAM-4I4O): RS-485 connector spacing
Parts:
- moved J2 3.76 mm to (164.0, 109.8)
- moved R1 3.50 mm to (167.8, 114.5)
- moved R2 3.50 mm to (164.0, 114.5)
- moved F2 3.20 mm to (157.9, 117.8)
Routing:
- net Net-(U2-A): track 18.1 -> 22.8 mm
- net Net-(D1-IN2): track 20.1 -> 23.6 mm
- net Net-(U2-B): track 11.9 -> 14.8 mm
- net Net-(D1-IN1): track 21.0 -> 24.0 mm
- net Net-(J9-Pin_1): track 3.75 -> 6.51 mm
- net Net-(U4-O1): track 18.5 -> 17.1 mm

Commit message: fix(LAM-4I4O): increase trace length to 0.5mm, fix missing ground trace for single-layer manufacturing
Routing:
- net Net-(J9-Pin_1): track 6.51 -> 5.08 mm
- net /OUT1: track 18.7 -> 19.8 mm
- net Net-(U4-O1): track 17.1 -> 16.3 mm

Commit message: add firmware
Parts:
- added REF**: 0x08_F_Cu, Logos:0x08_F_Cu, F.Cu at (120.0, 116.2)
Routing:
- net +5V: track 85.5 -> 83.8 mm
- net +12V: track 36.9 -> 35.9 mm
