File: LAM-4I4O/hardware/LAM-4I4O-REVC/LAM-4I4O-REVC.kicad_sch (KiCad schematic)
At the start: 39 parts, among them J1 MC1,5 2G-3.81, J2 MC1,5 2G-3.81, J3 MC1,5 2G-3.81, U1 CH32V003AxMx, U2 SN75176BDR, U3 LT1117-5.0

Commit message: fix(LAM-4I4O): incorrect PESD12VL2BT value in RS-485
Parts:
- D1: value PESD15VL2BT -> PESD12VL2BT; Manufacturer_Part_Number PESD15VS2UT,215 -> PESD12VL2BT,215; Mouser Part Number 771-PESD15VS2UT-T/R -> 771-PESD12VL2BT-T/R; Mouser Price/Stock https://www.mouser.co.uk/ProductDetail/Nexperia/PESD15VS2UT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 -> https://www.mouser.co.uk/ProductDetail/Nexperia/PESD12VL2BT
Changed lines of the file:
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@@
 		(fields_autoplaced yes)
 		(property "Reference" "D1"
-			(at 234.95 97.7899 90)
-			(effects
-				(font
-					(size 1.27 1.27)
-				)
-				(justify left)
-			)
-		)
-		(property "Value" "PESD15VL2BT"
-			(at 234.95 100.3299 90)
+			(at 234.95 97.79 90)
+			(effects
+				(font
+					(size 1.27 1.27)
+				)
+				(justify left)
+			)
+		)
+		(property "Value" "PESD12VL2BT"
+			(at 234.95 100.33 90)
 			(effects
 				(font
@@
 			)
 		)
-		(property "Datasheet" "https://assets.nexperia.com/documents/data-sheet/PESDXS2UT_SERIES.pdf"
+		(property "Datasheet" "https://assets.nexperia.com/documents/data-sheet/PESD12VL2BT.pdf"
 			(at 34.95 130.81 0)
 			(effects
@@
 			)
 		)
-		(property "Mouser Part Number" "771-PESD15VS2UT-T/R"
+		(property "Mouser Part Number" "771-PESD12VL2BT-T/R"
 			(at -265.05 130.81 0)
 			(effects
@@
 			)
 		)
-		(property "Mouser Price/Stock" "https://www.mouser.co.uk/ProductDetail/Nexperia/PESD15VS2UT215?qs=LOCUfHb8d9u9Mp9X1kxKXg%3D%3D"
+		(property "Mouser Price/Stock" "https://www.mouser.co.uk/ProductDetail/Nexperia/PESD12VL2BT"
 			(at -365.05 130.81 0)
 			(effects
@@
 			)
 		)
-		(property "Manufacturer_Part_Number" "PESD15VS2UT,215"
+		(property "Manufacturer_Part_Number" "PESD12VL2BT,215"
 			(at -565.05 130.81 0)
 			(effects
@@
 		)
 		(instances
-			(project "LAM-4I4O-REVB"
+			(project "LAM-4I4O-REVC"
 				(path "/d96e190f-efcd-4f25-974b-ce3a34276a2b"
 					(page "2")
