File: LAM-RPI-DMX/hardware/LAM-RPI-DMX/LAM-RPI-DMX.kicad_pcb (KiCad board)
At the start: 2 copper layers, 58.8 x 57.2 mm, 16 parts, among them J1 RPi GPIO Header, J2 PWR, J3 Conn_01x03_Socket, U1 DS1307Z+, U2 ADM3485EARZ, U3 Mini360, Y1 32.768K

Commit message: LAM-RPI-DMX: Revision A
Parts:
- moved R3 29.8 mm to (143.8, 86.0)
- moved U3 29.0 mm to (160.1, 107.0)
- moved BT1 18.0 mm to (158.2, 82.4), turned to -55 degrees
- moved Y1 11.2 mm to (138.2, 78.1), turned to 90 degrees
- moved C2 10.4 mm to (151.2, 96.1), turned to 180 degrees
- moved U1 10.1 mm to (130.8, 76.8), turned to 180 degrees
- moved R2 9.10 mm to (138.4, 95.9)
- moved TP2 9.10 mm to (134.9, 95.9)
- moved D1 9.10 mm to (131.4, 94.0)
- moved J2 9.10 mm to (126.7, 109.2)
- moved J3 9.10 mm to (126.7, 95.9)
- moved R1 9.10 mm to (138.4, 92.1)
- moved TP3 9.10 mm to (134.9, 92.1)
- moved U2 8.61 mm to (145.8, 93.6), turned to -90 degrees
Connections:
- J1 pad 8: /TX -> Net-(J1-UART_TX)
- R3 pad 1: /TX -> Net-(J1-UART_TX)
- R3 pad 2: Net-(U2-DI) -> /TX
- U2 pad 4: Net-(U2-DI) -> /TX
Routing:
- net Net-(J1-UART_TX): track 0.00 -> 56.5 mm
- net Net-(U2-DI): track 41.4 -> 0.00 mm
- net /TX: track 40.5 -> 3.70 mm
- net +3V3: track 43.3 -> 74.6 mm
- net +5V: track 70.6 -> 98.4 mm
- net Net-(J2-12V): track 16.0 -> 26.7 mm
- net Net-(BT1-+): track 28.7 -> 19.0 mm
- net /SDA: track 16.3 -> 6.73 mm
- net /SCL: track 15.1 -> 9.59 mm
- net Net-(U2-A): track 4.70 -> 7.91 mm
- net Net-(U2-B): track 11.7 -> 9.76 mm
- net Net-(U1-X2): track 4.39 -> 5.29 mm
- net Net-(U1-X1): track 4.41 -> 5.27 mm
- added copper zone on B.Cu, net GND
Other:
- board size 58.8 x 57.2 mm -> 55 x 58 mm
