File: LAM-RPI-DMX/hardware/LAM-RPI-DMX/LAM-RPI-DMX.kicad_sch (KiCad schematic)
At the start: 16 parts, among them J1 RPi GPIO Header, J2 PWR, J3 Conn_01x03_Socket, U1 DS1307Z+, U2 ADM3485EARZ, U3 Mini360, Y1 32.768K

Commit message: LAM-RPI-DMX: Revision A
Connections:
- net TX: now also R3.2, U2.4 (DI); no longer J1.8 (UART_TX), R3.1
- new net: J1.8 (UART_TX), R3.1
Changed lines of the file:
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@@
 	(wire
 		(pts
-			(xy 59.69 39.37) (xy 58.42 39.37)
+			(xy 71.12 39.37) (xy 68.58 39.37)
 		)
 		(stroke
@@
 	(wire
 		(pts
-			(xy 170.18 104.14) (xy 173.99 104.14)
+			(xy 177.8 104.14) (xy 184.15 104.14)
 		)
 		(stroke
@@
 	(wire
 		(pts
-			(xy 181.61 104.14) (xy 184.15 104.14)
+			(xy 60.96 39.37) (xy 58.42 39.37)
 		)
 		(stroke
@@
 	)
 	(label "TX"
-		(at 59.69 39.37 0)
+		(at 71.12 39.37 0)
 		(effects
 			(font
@@
 	)
 	(label "TX"
-		(at 170.18 104.14 180)
+		(at 177.8 104.14 180)
 		(effects
 			(font
@@
 	)
 	(symbol
+		(lib_id "Device:R")
+		(at 64.77 39.37 90)
+		(unit 1)
+		(exclude_from_sim no)
+		(in_bom yes)
+		(on_board yes)
+		(dnp no)
+		(fields_autoplaced yes)
+		(property "Reference" "R3"
+			(at 64.77 33.02 90)
+			(effects
+				(font
+					(size 1.27 1.27)
+				)
+			)
+		)
+		(property "Value" "0R"
+			(at 64.77 35.56 90)
+			(effects
+				(font
+					(size 1.27 1.27)
+				)
+			)
+		)
+		(property "Footprint" "Resistor_SMD:R_1206_3216Metric"
+			(at 64.77 41.148 90)
+			(effects
+				(font
+					(size 1.27 1.27)
+				)
+				(hide yes)
+			)
+		)
+		(property "Datasheet" "~"
+			(at 64.77 39.37 0)
+			(effects
+				(font
+					(size 1.27 1.27)
+				)
+				(hide yes)
+			)
+		)
+		(property "Description" "Resistor"
+			(at 64.77 39.37 0)
+			(effects
+				(font
+					(size 1.27 1.27)
+				)
+				(hide yes)
+			)
+		)
+		(pin "2"
+		)
+		(pin "1"
+		)
+		(instances
+			(project ""
+				(path "/30bb4d76-a899-42a0-a161-22b481828d6a"
+					(reference "R3")
+					(unit 1)
+				)
+			)
+		)
+	)
+	(symbol
 		(lib_id "power:GND")
 		(at 50.8 85.09 0)
@@
 					(unit 1)
 				)
-			)
-		)
-	)
-	(symbol
-		(lib_id "Device:R")
-		(at 177.8 104.14 90)
-		(mirror x)
-		(unit 1)
-		(exclude_from_sim no)
-		(in_bom yes)
-		(on_board yes)
-		(dnp no)
-		(property "Reference" "R3"
-			(at 177.8 110.49 90)
-			(effects
-				(font
-					(size 1.27 1.27)
-				)
-			)
-		)
-		(property "Value" "0R"
-			(at 177.8 107.95 90)
-			(effects
-				(font
-					(size 1.27 1.27)
-				)
-			)
-		)
-		(property "Footprint" "Resistor_SMD:R_1206_3216Metric"
-			(at 177.8 102.362 90)
-			(effects
-				(font
-					(size 1.27 1.27)
-				)
-				(hide yes)
-			)
-		)
-		(property "Datasheet" "~"
-			(at 177.8 104.14 0)
-			(effects
-				(font
-					(size 1.27 1.27)
-				)
-				(hide yes)
-			)
-		)
-		(property "Description" "Resistor"
-			(at 177.8 104.14 0)
-			(effects
-				(font
-					(size 1.27 1.27)
-				)
-				(hide yes)
-			)
-		)
-		(pin "2"
-		)
-		(pin "1"
-		)
-		(instances
-			(project ""
-				(path "/30bb4d76-a899-42a0-a161-22b481828d6a"
-					(reference "R3")
-					(unit 1)
-				)
