File: LAM-ZB-ROUTER/LAM-ZB-ROUTER.kicad_sch (KiCad schematic)
At the start: 12 parts, among them J1 PWR, J2 Conn_01x07_Pin, U1 CC2538, U2 LT1117-3.3

Commit message: LAM-ZB-ROUTER: Rev B
Parts:
- removed C6: 470uF / 25V, Capacitor_SMD:CP_Elec_6.3x5.9, symbol Device:C
- added C1: 100uF / 25V, Capacitor_THT:CP_Radial_D6.3mm_P2.50mm, symbol Device:C_Polarized
- added D3: RUN, LED_SMD:LED_1206_3216Metric, symbol Device:LED
- added R1: 270R, Resistor_SMD:R_0805_2012Metric, symbol Device:R
- added R2: 5K1, Resistor_SMD:R_0805_2012Metric, symbol Device:R
- added SW1: FLASH, Button_Switch_SMD:SW_Tactile_SPST_NO_Straight_CK_PTS636Sx25SMTRLFS, symbol Switch:SW_Push
Connections:
- net +12V: now also U2.3 (VI), C1.1; no longer U2.2 (VO)
- net +3V3: now also U2.2 (VO), SW1.2; no longer U2.3 (VI)
- net GND: now also C1.2, R1.1, R2.2
- net at U1.12 (PB1): now also D3.2 (A)
- net at U1.29 (PA7): now also R2.1, SW1.1
- new net: D3.1 (K), R1.2
- no-connect marks 25 -> 23
